File: Open Flight Controller.sch (EAGLE design)
At the start: 74 parts, among them IC1 TPS62133RGTT, IC2 LDL112PU33R, IC3 ICM-20689-V2.2, IC4 AK8963N, IC5 BMP280, IC6 STM32F765VGT6, Q1 IRLML6244TRPBF, Q2 SDTC114EET1G, X1 DM3BT-DSF-PEJS, X2 0473460001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

Commit message: Added reset-pin and pwm-led
Parts:
- added D4, D5: RBR3MM40ATR, RBR3MM40ATR:RBR3MM40ATR
- added LED3: BLUE, VLMB1300-GS08:VLMB1300-GS08
- added Q3: SDTC114EET1G, SDTC114EET1G:SDTC114EET1G
- added R12: 1k, CRCW06031K00FKEA:CRCW06031K00FKEA
- SV9: value MA03-2 -> (none); device MA03-2:MA03-2 -> MA04-2:MA04-2
Connections:
- net GPIO2(P+T_CS) renamed GPIO2
- new net BOOT_PIN: D5.A, SV9.7
- new net N$17: Q3.E, R12.2
- new net N$20: LED3.A, R12.1
- new net RST_PIN: D4.A, SV9.8
- net !RST: now also D4.C
- net 3.3V: now also Q3.C
- net BOOT: now also D5.C
- net GND: now also LED3.K
- net PWM14/LCD_CLK: now also Q3.B
Changed lines of the file:
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@@
 <?xml version="1.0" encoding="utf-8"?>
 <!DOCTYPE eagle SYSTEM "eagle.dtd">
-<eagle version="9.0.1">
+<eagle version="9.0.0">
 <drawing>
 <settings>
@@
 <part name="GND51" library="supply1" library_urn="urn:adsk.eagle:library:371" deviceset="GND" device=""/>
 <part name="GND52" library="supply1" library_urn="urn:adsk.eagle:library:371" deviceset="GND" device=""/>
-<part name="SV9" library="MA03-2" deviceset="MA03-2" device=""/>
+<part name="SV9" library="MA04-2" deviceset="MA04-2" device="" package3d_urn="urn:adsk.eagle:package:8368/1"/>
 <part name="SV10" library="MA03-2" deviceset="MA03-2" device=""/>
 <part name="SV11" library="MA03-2" deviceset="MA03-2" device=""/>
@@
 <part name="GND55" library="supply1" library_urn="urn:adsk.eagle:library:371" deviceset="GND" device=""/>
 <part name="C25" library="GRM188R71H104KA93D" deviceset="GRM188R71H104KA93D" device="" value="0.1uF"/>
+<part name="LED3" library="VLMB1300-GS08" deviceset="VLMB1300-GS08" device="" value="BLUE"/>
+<part name="Q3" library="SDTC114EET1G" deviceset="SDTC114EET1G" device=""/>
+<part name="R12" library="CRCW06031K00FKEA" deviceset="CRCW06031K00FKEA" device="" value="1k"/>
+<part name="GND56" library="supply1" library_urn="urn:adsk.eagle:library:371" deviceset="GND" device=""/>
+<part name="D4" library="RBR3MM40ATR" deviceset="RBR3MM40ATR" device="" value=""/>
+<part name="D5" library="RBR3MM40ATR" deviceset="RBR3MM40ATR" device="" value=""/>
 </parts>
 <sheets>
@@
 <segment>
 <pinref part="SV9" gate="G$1" pin="1"/>
-<wire x1="254" y1="91.44" x2="259.08" y2="91.44" width="0.1524" layer="91"/>
-<label x="261.62" y="91.44" size="1.778" layer="95"/>
+<wire x1="254" y1="88.9" x2="259.08" y2="88.9" width="0.1524" layer="91"/>
+<label x="261.62" y="88.9" size="1.778" layer="95"/>
 </segment>
 </net>
@@
 <segment>
 <pinref part="SV9" gate="G$1" pin="6"/>
-<wire x1="238.76" y1="96.52" x2="233.68" y2="96.52" width="0.1524" layer="91"/>
-<label x="198.12" y="96.52" size="1.778" layer="95"/>
+<wire x1="238.76" y1="93.98" x2="233.68" y2="93.98" width="0.1524" layer="91"/>
+<label x="198.12" y="93.98" size="1.778" layer="95"/>
 </segment>
 </net>
@@
 <segment>
 <pinref part="SV9" gate="G$1" pin="5"/>
-<wire x1="254" y1="96.52" x2="259.08" y2="96.52" width="0.1524" layer="91"/>
-<label x="261.62" y="96.52" size="1.778" layer="95"/>
+<wire x1="254" y1="93.98" x2="259.08" y2="93.98" width="0.1524" layer="91"/>
+<label x="261.62" y="93.98" size="1.778" layer="95"/>
 </segment>
 </net>
@@
 <segment>
 <pinref part="SV9" gate="G$1" pin="3"/>
-<wire x1="254" y1="93.98" x2="259.08" y2="93.98" width="0.1524" layer="91"/>
-<label x="261.62" y="93.98" size="1.778" layer="95"/>
+<wire x1="254" y1="91.44" x2="259.08" y2="91.44" width="0.1524" layer="91"/>
+<label x="261.62" y="91.44" size="1.778" layer="95"/>
 </segment>
 </net>
@@
 <segment>
 <pinref part="SV9" gate="G$1" pin="4"/>
-<wire x1="238.76" y1="93.98" x2="233.68" y2="93.98" width="0.1524" layer="91"/>
-<label x="198.12" y="93.98" size="1.778" layer="95"/>
+<wire x1="238.76" y1="91.44" x2="233.68" y2="91.44" width="0.1524" layer="91"/>
+<label x="198.12" y="91.44" size="1.778" layer="95"/>
 </segment>
 </net>
@@
 <segment>
 <pinref part="SV9" gate="G$1" pin="2"/>
-<wire x1="238.76" y1="91.44" x2="233.68" y2="91.44" width="0.1524" layer="91"/>
-<label x="198.12" y="91.44" size="1.778" layer="95"/>
+<wire x1="238.76" y1="88.9" x2="233.68" y2="88.9" width="0.1524" layer="91"/>
+<label x="198.12" y="88.9" size="1.778" layer="95"/>
 </segment>
 </net>
@@
 </segment>
 </net>
+<net name="RST_PIN" class="0">
+<segment>
+<pinref part="SV9" gate="G$1" pin="8"/>
+<wire x1="238.76" y1="96.52" x2="233.68" y2="96.52" width="0.1524" layer="91"/>
+<label x="198.12" y="96.52" size="1.778" layer="95"/>
+</segment>
+</net>
+<net name="BOOT_PIN" class="0">
+<segment>
+<pinref part="SV9" gate="G$1" pin="7"/>
+<wire x1="254" y1="96.52" x2="259.08" y2="96.52" width="0.1524" layer="91"/>
+<label x="261.62" y="96.52" size="1.778" layer="95"/>
+</segment>
+</net>
 </nets>
 </sheet>
@@
 <instance part="GND55" gate="1" x="81.28" y="83.82"/>
 <instance part="C25" gate="G$1" x="81.28" y="93.98"/>
+<instance part="LED3" gate="G$1" x="325.12" y="119.38" rot="R90"/>
+<instance part="Q3" gate="G$1" x="289.56" y="147.32"/>
+<instance part="R12" gate="G$1" x="312.42" y="119.38" rot="R90"/>
+<instance part="GND56" gate="1" x="325.12" y="114.3"/>
+<instance part="D4" gate="G$1" x="289.56" y="205.74" rot="R270"/>
+<instance part="D5" gate="G$1" x="330.2" y="226.06" rot="R270"/>
 </instances>
 <busses>
@@
 <wire x1="81.28" y1="86.36" x2="81.28" y2="88.9" width="0.1524" layer="91"/>
 </segment>
+<segment>
+<pinref part="GND56" gate="1" pin="GND"/>
+<pinref part="LED3" gate="G$1" pin="K"/>
+<wire x1="325.12" y1="116.84" x2="325.12" y2="114.3" width="0.1524" layer="91"/>
+<wire x1="325.12" y1="116.84" x2="325.12" y2="119.38" width="0.1524" layer="91"/>
+</segment>
 </net>
 <net name="3.3V" class="0">
@@
 <label x="81.28" y="236.22" size="1.778" layer="95" rot="R90" xref="yes"/>
 </segment>
+<segment>
+<pinref part="Q3" gate="G$1" pin="C"/>
+<wire x1="309.88" y1="152.4" x2="312.42" y2="152.4" width="0.1524" layer="91"/>
+<wire x1="312.42" y1="152.4" x2="312.42" y2="157.48" width="0.1524" layer="91"/>
+<label x="312.42" y="157.48" size="1.778" layer="95" rot="R90" xref="yes"/>
+</segment>
 </net>
 <net name="N$10" class="0">
@@
 <pinref part="S1" gate="G$1" pin="NO_1"/>
 <wire x1="330.2" y1="218.44" x2="325.12" y2="218.44" width="0.1524" layer="91"/>
+<pinref part="D5" gate="G$1" pin="C"/>
+<wire x1="330.2" y1="223.52" x2="330.2" y2="218.44" width="0.1524" layer="91"/>
 </segment>
 </net>
@@
 </segment>
 </net>
-<net name="GPIO2(P+T_CS)" class="0">
+<net name="GPIO2" class="0">
 <segment>
 <pinref part="IC6" gate="G$1" pin="PE4"/>
@@
 <label x="25.4" y="119.38" size="1.778" layer="95"/>
 </segment>
+<segment>
+<pinref part="Q3" gate="G$1" pin="B"/>
+<wire x1="289.56" y1="147.32" x2="284.48" y2="147.32" width="0.1524" layer="91"/>
+<label x="261.62" y="147.32" size="1.778" layer="95"/>
+</segment>
 </net>
 <net name="USART3_TX" class="0">
@@
 <wire x1="276.86" y1="198.12" x2="281.94" y2="198.12" width="0.1524" layer="91"/>
 <pinref part="R11" gate="G$1" pin="1"/>
-<wire x1="281.94" y1="198.12" x2="287.02" y2="198.12" width="0.1524" layer="91"/>
+<wire x1="281.94" y1="198.12" x2="289.56" y2="198.12" width="0.1524" layer="91"/>
+<wire x1="289.56" y1="198.12" x2="294.64" y2="198.12" width="0.1524" layer="91"/>
 <wire x1="281.94" y1="198.12" x2="281.94" y2="200.66" width="0.1524" layer="91"/>
 <junction x="281.94" y="198.12"/>
-<label x="289.56" y="198.12" size="1.778" layer="95"/>
+<label x="297.18" y="198.12" size="1.778" layer="95"/>
 <pinref part="S2" gate="G$1" pin="P$2"/>
+<pinref part="D4" gate="G$1" pin="C"/>
+<wire x1="289.56" y1="203.2" x2="289.56" y2="198.12" width="0.1524" layer="91"/>
+<junction x="289.56" y="198.12"/>
 </segment>
 </net>
@@
 </segment>
 </net>
+<net name="N$17" class="0">
+<segment>
+<pinref part="Q3" gate="G$1" pin="E"/>
+<pinref part="R12" gate="G$1" pin="2"/>
+<wire x1="309.88" y1="137.16" x2="312.42" y2="137.16" width="0.1524" layer="91"/>
+<wire x1="312.42" y1="137.16" x2="312.42" y2="132.08" width="0.1524" layer="91"/>
+</segment>
+</net>
+<net name="N$20" class="0">
+<segment>
+<pinref part="R12" gate="G$1" pin="1"/>
+<wire x1="312.42" y1="119.38" x2="312.42" y2="114.3" width="0.1524" layer="91"/>
+<wire x1="312.42" y1="114.3" x2="317.5" y2="114.3" width="0.1524" layer="91"/>
+<wire x1="317.5" y1="114.3" x2="317.5" y2="137.16" width="0.1524" layer="91"/>
+<pinref part="LED3" gate="G$1" pin="A"/>
+<wire x1="317.5" y1="137.16" x2="325.12" y2="137.16" width="0.1524" layer="91"/>
+<wire x1="325.12" y1="137.16" x2="325.12" y2="129.54" width="0.1524" layer="91"/>
+</segment>
+</net>
+<net name="RST_PIN" class="0">
+<segment>
+<pinref part="D4" gate="G$1" pin="A"/>
+<wire x1="289.56" y1="208.28" x2="289.56" y2="215.9" width="0.1524" layer="91"/>
+<label x="289.56" y="215.9" size="1.778" layer="95" rot="R90" xref="yes"/>
+</segment>
+</net>
+<net name="BOOT_PIN" class="0">
+<segment>
+<pinref part="D5" gate="G$1" pin="A"/>
+<wire x1="330.2" y1="228.6" x2="330.2" y2="233.68" width="0.1524" layer="91"/>
+<label x="330.2" y="233.68" size="1.778" layer="95" rot="R90" xref="yes"/>
+</segment>
+</net>
 </nets>
 </sheet>
@@
 will not be understood (or retained) with this version.
 </note>
+<note version="8.3" severity="warning">
+Since Version 8.3, EAGLE supports the association of 3D packages
+with devices in libraries, schematics, and board files. Those 3D
+packages will not be understood (or retained) with this version.
+</note>
 </compatibility>
